Commit message: Edit navigation stack configurations

File: sphinx_description/urdf/hokuyo.urdf.xacro (robot description, xacro)
@@ -3,9 +3,11 @@
     <!-- SENSORS -->
       <!-- hokuyo --> -->
+      <xacro:property name="hokuyo_mesh_link" value="package://sphinx_description/meshes/hokuyo.dae" />
+      <xacro:property name="hokuyo_mesh_scale" value="1.0" />
       <link name="hokuyo_link">
         <visual>
           <origin rpy="0 0 0" xyz="0 0 0"/>
           <geometry>
-            <box size="0.02 0.02 0.02"/>
+            <mesh filename="${hokuyo_mesh_link}" scale="${hokuyo_mesh_scale} ${hokuyo_mesh_scale} ${hokuyo_mesh_scale}"/>
           </geometry>
           <material name="Blue"/>
@@ -23,32 +25,9 @@
       <child link="hokuyo_link"/>
     </joint>
-  <!-- hokuyo Mesh file--> -->
-  <xacro:property name="hokuyo_mesh_link" value="package://sphinx_description/meshes/hokuyo.dae" />
-  <xacro:property name="hokuyo_mesh_scale" value="1.0" />
-  <link name="hokuyo_mesh_link">
-    <visual>
-      <origin rpy="0 0 0" xyz="0 0 0"/>
-      <geometry>
-        <mesh filename="${hokuyo_mesh_link}" scale="${hokuyo_mesh_scale} ${hokuyo_mesh_scale} ${hokuyo_mesh_scale}"/>
-      </geometry>
-      <material name="Blue"/>
-    </visual>
-    <collision>
-        <origin rpy="0 0 0" xyz="0 0 0"/>
-        <geometry>
-            <mesh filename="${hokuyo_mesh_link}" scale="${hokuyo_mesh_scale} ${hokuyo_mesh_scale} ${hokuyo_mesh_scale}"/>
-        </geometry>
-    </collision>
-  </link>
-  <joint name="hokuyo_mesh_joint" type="fixed">
-    <origin rpy="0 0 0" xyz="0.15 0 0.12"/>
-    <parent link="base_link"/>
-    <child link="hokuyo_mesh_link"/>
-  </joint>
   <gazebo reference="hokuyo_link">
     <material>Gazebo/Blue</material>
     <turnGravityOff>false</turnGravityOff>
     <sensor name="head_hokuyo_sensor" type="ray">
-      <pose>0.025 0 0 0 0 0</pose>
+      <pose>0.15 0 0.12 0 0 0</pose>
       <visualize>false</visualize>
       <update_rate>40</update_rate>
@@ -69,5 +48,5 @@
       </ray>
       <plugin filename="libgazebo_ros_laser.so" name="gazebo_ros_head_hokuyo_controller">
-        <topicName>/scan</topicName>
+        <topicName>laser/scan</topicName>
         <frameName>hokuyo_link</frameName>
       </plugin>
